File: touchcard/touchcard.kicad_pcb (KiCad board)
At the start: 2 copper layers, 85 x 55 mm, 15 parts, among them J1 Conn_01x04, J2 USB_C_Receptacle_USB2.0, U1 STM32F042K6Tx, U2 USBLC6-2SC6, U3 AP1117-33

Commit message: PCB Review
Routing:
- net +3V3: track 69.7 -> 77.0 mm
- net +5V: track 38.1 -> 39.8 mm
- net GND: track 26.5 -> 27.3 mm, vias 55 -> 59
Other:
- board text added: "contact@synthron.de"
