File: touchcard/touchcard.kicad_sch (KiCad schematic)
At the start: 14 parts, among them J1 Conn_01x04, J2 USB_C_Receptacle_USB2.0, U1 STM32F042K6Tx, U2 USBLC6-2SC6, U3 AP1117-33

Commit message: Finalize Schematic and Layout
Parts:
- removed R3: 10k, eigene:0603_1608Metric_Pad1.08x0.95mm_MidMount, symbol Device:R
Connections:
- net DP: now also U2.6 (I/O1); no longer U2.1 (I/O1)
- net USB_DP: now also U2.1 (I/O1); no longer U2.6 (I/O1)
- net DM renamed DN
- net DN: now also U2.4 (I/O2); no longer U2.3 (I/O2)
- net USB_DM renamed USB_DN
- net USB_DN: now also U2.3 (I/O2); no longer U2.4 (I/O2)
- no-connect marks 8 -> 9
Other:
- moved on the sheet: U2
Changed lines of the file:
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@@
   )
   (no_connect (at 63.5 92.71))
+  (no_connect (at 63.5 80.01))
   (no_connect (at 63.5 118.11))
   (no_connect (at 63.5 113.03))
@@
     (stroke (width 0) (type default))
   )
-  (wire (pts (xy 50.8 78.74) (xy 50.8 80.01))
-    (stroke (width 0) (type default))
-  )
   (wire (pts (xy 218.44 120.65) (xy 218.44 121.92))
     (stroke (width 0) (type default))
@@
     (stroke (width 0) (type default))
   )
-  (wire (pts (xy 142.24 100.33) (xy 144.78 100.33))
+  (wire (pts (xy 167.64 100.33) (xy 165.1 100.33))
     (stroke (width 0) (type default))
   )
@@
     (stroke (width 0) (type default))
   )
-  (wire (pts (xy 60.96 80.01) (xy 63.5 80.01))
-    (stroke (width 0) (type default))
-  )
   (wire (pts (xy 73.66 74.93) (xy 73.66 72.39))
     (stroke (width 0) (type default))
@@
     (stroke (width 0) (type default))
   )
-  (wire (pts (xy 165.1 100.33) (xy 167.64 100.33))
+  (wire (pts (xy 144.78 100.33) (xy 142.24 100.33))
     (stroke (width 0) (type default))
   )
@@
   )
   (wire (pts (xy 73.66 72.39) (xy 76.2 72.39))
-    (stroke (width 0) (type default))
-  )
-  (wire (pts (xy 50.8 80.01) (xy 53.34 80.01))
     (stroke (width 0) (type default))
   )
@@
     (effects (font (size 1.27 1.27)) (justify right bottom))
   )
-  (label "DM" (at 179.07 96.52 0) (fields_autoplaced)
+  (label "DN" (at 179.07 96.52 0) (fields_autoplaced)
     (effects (font (size 1.27 1.27)) (justify left bottom))
   )
-  (label "USB_DM" (at 121.92 96.52 0) (fields_autoplaced)
+  (label "USB_DN" (at 121.92 96.52 0) (fields_autoplaced)
     (effects (font (size 1.27 1.27)) (justify left bottom))
   )
@@
     )
   )
-  (symbol (lib_id "power:+5V") (at 142.24 100.33 90) (unit 1)
-    (in_bom yes) (on_board yes) (dnp no) (fields_autoplaced)
-    (property "Reference" "#PWR06" (at 146.05 100.33 0)
-      (effects (font (size 1.27 1.27)) hide)
-    )
-    (property "Value" "+5V" (at 139.0651 100.6468 90)
-      (effects (font (size 1.27 1.27)) (justify left))
-    )
-    (property "Footprint" "" (at 142.24 100.33 0)
-      (effects (font (size 1.27 1.27)) hide)
-    )
-    (property "Datasheet" "" (at 142.24 100.33 0)
+  (symbol (lib_id "power:+5V") (at 167.64 100.33 270) (mirror x) (unit 1)
+    (in_bom yes) (on_board yes) (dnp no) (fields_autoplaced)
+    (property "Reference" "#PWR06" (at 163.83 100.33 0)
+      (effects (font (size 1.27 1.27)) hide)
+    )
+    (property "Value" "+5V" (at 170.8149 100.6468 90)
+      (effects (font (size 1.27 1.27)) (justify left))
+    )
+    (property "Footprint" "" (at 167.64 100.33 0)
+      (effects (font (size 1.27 1.27)) hide)
+    )
+    (property "Datasheet" "" (at 167.64 100.33 0)
       (effects (font (size 1.27 1.27)) hide)
     )
@@
         (path "/3cd4ffe4-2818-4a73-988c-23c4068d93a0"
           (reference "C1") (unit 1)
-        )
-      )
-    )
-  )
-  (symbol (lib_id "power:+3V3") (at 50.8 78.74 0) (unit 1)
-    (in_bom yes) (on_board yes) (dnp no) (fields_autoplaced)
-    (property "Reference" "#PWR014" (at 50.8 82.55 0)
-      (effects (font (size 1.27 1.27)) hide)
-    )
-    (property "Value" "+3V3" (at 50.8 75.2381 0)
-      (effects (font (size 1.27 1.27)))
-    )
-    (property "Footprint" "" (at 50.8 78.74 0)
-      (effects (font (size 1.27 1.27)) hide)
-    )
-    (property "Datasheet" "" (at 50.8 78.74 0)
-      (effects (font (size 1.27 1.27)) hide)
-    )
-    (pin "1")
-    (instances
-      (project "touchcard"
-        (path "/3cd4ffe4-2818-4a73-988c-23c4068d93a0"
-          (reference "#PWR014") (unit 1)
         )
       )
@@
     )
   )
-  (symbol (lib_id "Power_Protection:USBLC6-2SC6") (at 154.94 100.33 90) (unit 1)
+  (symbol (lib_id "Power_Protection:USBLC6-2SC6") (at 154.94 100.33 270) (mirror x) (unit 1)
     (in_bom yes) (on_board yes) (dnp no)
-    (property "Reference" "U2" (at 166.37 104.14 90)
-      (effects (font (size 1.27 1.27)) (justify left))
-    )
-    (property "Value" "USBLC6-2SC6" (at 176.53 106.68 90)
-      (effects (font (size 1.27 1.27)) (justify left))
-    )
-    (property "Footprint" "eigene:SOT-23-6_MidMount" (at 167.64 100.33 0)
-      (effects (font (size 1.27 1.27)) hide)
-    )
-    (property "Datasheet" "https://www.st.com/resource/en/datasheet/usblc6-2.pdf" (at 146.05 95.25 0)
+    (property "Reference" "U2" (at 162.56 104.14 90)
+      (effects (font (size 1.27 1.27)) (justify left))
+    )
+    (property "Value" "USBLC6-2SC6" (at 162.56 107.95 90)
+      (effects (font (size 1.27 1.27)) (justify left))
+    )
+    (property "Footprint" "eigene:SOT-23-6_MidMount" (at 142.24 100.33 0)
+      (effects (font (size 1.27 1.27)) hide)
+    )
+    (property "Datasheet" "https://www.st.com/resource/en/datasheet/usblc6-2.pdf" (at 163.83 95.25 0)
       (effects (font (size 1.27 1.27)) hide)
     )
@@
         (path "/3cd4ffe4-2818-4a73-988c-23c4068d93a0"
           (reference "R2") (unit 1)
-        )
-      )
-    )
-  )
-  (symbol (lib_id "Device:R") (at 57.15 80.01 90) (unit 1)
-    (in_bom yes) (on_board yes) (dnp no) (fields_autoplaced)
-    (property "Reference" "R3" (at 57.15 75.9841 90)
-      (effects (font (size 1.27 1.27)))
-    )
-    (property "Value" "10k" (at 57.15 77.9051 90)
-      (effects (font (size 1.27 1.27)))
-    )
-    (property "Footprint" "eigene:0603_1608Metric_Pad1.08x0.95mm_MidMount" (at 57.15 81.788 90)
-      (effects (font (size 1.27 1.27)) hide)
-    )
-    (property "Datasheet" "~" (at 57.15 80.01 0)
-      (effects (font (size 1.27 1.27)) hide)
-    )
-    (pin "1")
-    (pin "2")
-    (instances
-      (project "touchcard"
-        (path "/3cd4ffe4-2818-4a73-988c-23c4068d93a0"
-          (reference "R3") (unit 1)
         )
       )
@@
     )
   )
-  (symbol (lib_id "power:GND") (at 167.64 100.33 90) (unit 1)
-    (in_bom yes) (on_board yes) (dnp no) (fields_autoplaced)
-    (property "Reference" "#PWR05" (at 173.99 100.33 0)
-      (effects (font (size 1.27 1.27)) hide)
-    )
-    (property "Value" "GND" (at 170.815 100.6468 90)
+  (symbol (lib_id "power:GND") (at 142.24 100.33 270) (mirror x) (unit 1)
+    (in_bom yes) (on_board yes) (dnp no) (fields_autoplaced)
+    (property "Reference" "#PWR05" (at 135.89 100.33 0)
+      (effects (font (size 1.27 1.27)) hide)
+    )
+    (property "Value" "GND" (at 139.065 100.6468 90)
       (effects (font (size 1.27 1.27)) (justify right))
     )
-    (property "Footprint" "" (at 167.64 100.33 0)
-      (effects (font (size 1.27 1.27)) hide)
-    )
-    (property "Datasheet" "" (at 167.64 100.33 0)
-      (effects (font (size 1.27 1.27)) hide)
-    )
+    (property "Footprint" "" (at 142.24 100.33 0)
+      (effects (font (size 1.27 1.27)) hide)
+    )
+    (property "Datasheet" "" (at 142.24 100.33 0)
+      (effects (font (size 1.27 1.27)) hide)
+    )
